File: FT4232HP/uart-to-usb.kicad_sch (KiCad schematic)
At the start: 16 parts, among them J1 USB_C_Receptacle_USB2.0_16P, J2 Conn_01x05_Socket, SW1 SW_Push, U1 FT4232H, U2 AP2112K-3.3, Y1 12MHz

Commit message: Finish 4232 routing
Parts:
- J2: value Conn_01x05_Socket -> Conn_01x04_Pin; footprint Connector_JST:JST_XH_S5B-XH-A_1x05_P2.50mm_Horizontal -> Connector_JST:JST_XH_S4B-XH-A_1x04_P2.50mm_Horizontal; symbol Connector:Conn_01x05_Socket -> Connector:Conn_01x04_Pin; LCSC (none) -> C157925
Connections:
- net GND: now also J2.4 (Pin_4); no longer J2.5 (Pin_5)
- net MCU_TX_D: no longer names the net of U1.52 (DDBUS1)
- net MCU_TX_D: no longer J2.4 (Pin_4)
Other:
- moved on the sheet: J2
Changed lines of the file:
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@@
-	(wire
-		(pts
-			(xy 247.65 50.8) (xy 259.08 50.8)
-		)
-		(stroke
-			(width 0)
-			(type default)
-		)
-	)
 	(wire
 		(pts
@@
 	(wire
 		(pts
-			(xy 247.65 48.26) (xy 259.08 48.26)
+			(xy 247.65 50.8) (xy 265.43 50.8)
 		)
 		(stroke
@@
 	(wire
 		(pts
+			(xy 265.43 53.34) (xy 259.08 53.34)
+		)
+		(stroke
+			(width 0)
+			(type default)
+		)
+	)
+	(wire
+		(pts
 			(xy 72.39 62.23) (xy 81.28 62.23)
 		)
@@
 	(wire
 		(pts
-			(xy 214.63 111.76) (xy 219.71 111.76)
-		)
-		(stroke
-			(width 0)
-			(type default)
-		)
-	)
-	(wire
-		(pts
 			(xy 147.32 45.72) (xy 153.67 45.72)
 		)
@@
 	(wire
 		(pts
+			(xy 247.65 48.26) (xy 265.43 48.26)
+		)
+		(stroke
+			(width 0)
+			(type default)
+		)
+	)
+	(wire
+		(pts
 			(xy 196.85 25.4) (xy 196.85 29.21)
 		)
@@
 	(wire
 		(pts
-			(xy 247.65 45.72) (xy 259.08 45.72)
-		)
-		(stroke
-			(width 0)
-			(type default)
-		)
-	)
-	(wire
-		(pts
 			(xy 146.05 129.54) (xy 153.67 129.54)
 		)
@@
 	(wire
 		(pts
-			(xy 247.65 43.18) (xy 259.08 43.18)
+			(xy 247.65 45.72) (xy 265.43 45.72)
 		)
 		(stroke
@@
 	)
 	(label "MCU_TX_A"
-		(at 247.65 43.18 0)
+		(at 247.65 45.72 0)
 		(effects
 			(font
@@
 	)
 	(label "MCU_TX_B"
-		(at 247.65 45.72 0)
+		(at 247.65 48.26 0)
 		(effects
 			(font
@@
 		)
 	)
-	(label "MCU_TX_D"
-		(at 247.65 50.8 0)
-		(effects
-			(font
-				(size 1.27 1.27)
-			)
-			(justify left bottom)
-		)
-	)
 	(label "SBU1"
 		(at 67.31 102.87 0)
@@
 		)
 	)
-	(label "MCU_TX_D"
-		(at 219.71 111.76 0)
-		(effects
-			(font
-				(size 1.27 1.27)
-			)
-			(justify left bottom)
-		)
-	)
 	(label "MCU_TX_C"
-		(at 247.65 48.26 0)
+		(at 247.65 50.8 0)
 		(effects
 			(font
@@
 	)
 	(symbol
-		(lib_id "Connector:Conn_01x05_Socket")
-		(at 264.16 48.26 0)
+		(lib_id "Connector:Conn_01x04_Pin")
+		(at 270.51 48.26 0)
+		(mirror y)
 		(unit 1)
 		(body_style 1)
@@
 		(in_pos_files yes)
 		(dnp no)
-		(fields_autoplaced yes)
 		(property "Reference" "J2"
-			(at 265.43 46.9899 0)
-			(show_name no)
-			(do_not_autoplace no)
-			(effects
-				(font
-					(size 1.27 1.27)
-				)
-				(justify left)
-			)
-		)
-		(property "Value" "Conn_01x05_Socket"
-			(at 265.43 49.5299 0)
-			(show_name no)
-			(do_not_autoplace no)
-			(effects
-				(font
-					(size 1.27 1.27)
-				)
-				(justify left)
-			)
-		)
-		(property "Footprint" "Connector_JST:JST_XH_S5B-XH-A_1x05_P2.50mm_Horizontal"
-			(at 264.16 48.26 0)
+			(at 269.875 40.64 0)
+			(show_name no)
+			(do_not_autoplace no)
+			(effects
+				(font
+					(size 1.27 1.27)
+				)
+			)
+		)
+		(property "Value" "Conn_01x04_Pin"
+			(at 269.875 43.18 0)
+			(show_name no)
+			(do_not_autoplace no)
+			(effects
+				(font
+					(size 1.27 1.27)
+				)
+			)
+		)
+		(property "Footprint" "Connector_JST:JST_XH_S4B-XH-A_1x04_P2.50mm_Horizontal"
+			(at 270.51 48.26 0)
 			(hide yes)
 			(show_name no)
@@
 		)
 		(property "Datasheet" ""
-			(at 264.16 48.26 0)
+			(at 270.51 48.26 0)
 			(hide yes)
 			(show_name no)
@@
 		)
 		(property "Description" "Generic connector, single row, 01x05, script generated"
-			(at 264.16 48.26 0)
+			(at 270.51 48.26 0)
+			(hide yes)
+			(show_name no)
+			(do_not_autoplace no)
+			(effects
+				(font
+					(size 1.27 1.27)
+				)
+			)
+		)
+		(property "LCSC" "C157925"
+			(at 270.51 48.26 0)
 			(hide yes)
 			(show_name no)
@@
 		(pin "4"
 		)
-		(pin "5"
-		)
 		(instances
